Commit message: Update demo

File: demo/assets/urdf/garmi.urdf (robot description, URDF)
Before this commit: robot r100-0603, 64 links, 63 joints
Links:
- link arm_0_fr3_link0: geometry 
- link arm_0_fr3_link1: geometry 
- link arm_0_fr3_link2: geometry 
- link arm_0_fr3_link3: geometry 
- link arm_0_fr3_link4: geometry 
- link arm_0_fr3_link5: geometry 
- link arm_0_fr3_link6: geometry 
- link arm_0_fr3_link7: geometry 
- link arm_0_gripper_fr3_hand: geometry 
- link arm_0_gripper_fr3_leftfinger: geometry 
- link arm_0_gripper_fr3_rightfinger: geometry 
- link arm_1_fr3_link0: geometry 
- link arm_1_fr3_link1: geometry 
- link arm_1_fr3_link2: geometry 
- link arm_1_fr3_link3: geometry 
- link arm_1_fr3_link4: geometry 
- link arm_1_fr3_link5: geometry 
- link arm_1_fr3_link6: geometry 
- link arm_1_fr3_link7: geometry 
- link arm_1_gripper_fr3_hand: geometry 
- link arm_1_gripper_fr3_leftfinger: geometry 
- link arm_1_gripper_fr3_rightfinger: geometry 
- link axle_link: geometry 
- link body_link: geometry 
- link chassis_link: geometry 
- link cover_link: geometry 
- link front_cover_link: geometry 
- link front_left_wheel_link: geometry 
- link front_lights_link: geometry 
- link front_right_wheel_link: geometry 
- link front_rocker_link: geometry 
- link head: geometry 
- link imu_1_link: geometry 
- link left_side_cover_link: geometry 
- link lidar2d_0_link: geometry 
- link lidar2d_1_link: geometry 
- link lift_0_base_link: geometry 
- link lift_0_lower_link: geometry 
- link lift_0_plate_link: geometry 
- link lift_0_upper_link: geometry 
- link mounting_plate_link: geometry 
- link neck_1: geometry 
- link neck_2: geometry 
- link rear_cover_link: geometry 
- link rear_left_wheel_link: geometry 
- link rear_lights_link: geometry 
- link rear_right_wheel_link: geometry 
- link rear_rocker_link: geometry 
- link right_side_cover_link: geometry 
- link riser_link: geometry 
Joints:
- joint arm_0_gripper_fr3_finger_joint2: mimic joint=arm_0_gripper_fr3_finger_joint1 -> (none)
- joint arm_1_gripper_fr3_finger_joint2: mimic joint=arm_1_gripper_fr3_finger_joint1 -> (none)
- joint lift_0_upper_joint: mimic joint=lift_0_lower_joint -> (none)
